File: src/soldering_is_easy.brd (EAGLE design)
At the start: 38.2 x 61.5 mm, 3 parts

Commit message: rev 1.1
Parts:
- moved BATTERY_1 3.09 mm to (28.1, 16.0)
Routing:
- net N$3: track 46.9 -> 49.6 mm
- net N$1: track 50.1 -> 52.3 mm
Other:
- board text added: "Soldering is easy rev 1.1"
- board text removed: "Build Brighton www.buildbrighton.com"
- board text removed: "Soldering is easy rev 1.0"
Changed lines of the file:
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@@
 <rectangle x1="8.339275" y1="7.214175" x2="8.485325" y2="7.220525" layer="21"/>
 <text x="9.75" y="20.25" size="1.4224" layer="22" font="vector" ratio="9" rot="MR0" align="top-right">Battery Holder</text>
-<text x="4.75" y="33.25" size="2.54" layer="21" font="vector">I CAN SOLDER!</text>
+<text x="4.75" y="32.5" size="2.54" layer="21" font="vector">I CAN SOLDER!</text>
 <text x="11.25" y="6.75" size="0.8128" layer="21" font="vector">Designed by Justin Nel</text>
 <text x="11.25" y="2.75" size="1" layer="21" font="vector">[ www.cyber-lane.com ]</text>
-<text x="1.25" y="29.75" size="1.016" layer="21" font="fixed" rot="R270">Soldering is easy rev 1.0</text>
-<text x="33.5" y="28" size="1.016" layer="21" font="fixed" rot="R90" align="bottom-right">Build Brighton
-www.buildbrighton.com</text>
+<text x="1.25" y="29.75" size="1.016" layer="21" font="fixed" rot="R270">Soldering is easy rev 1.1</text>
 <rectangle x1="-0.5" y1="30" x2="37.5" y2="36" layer="40"/>
 <text x="25.5" y="32" size="1.778" layer="22" rot="MR0">Place Pin Here:</text>
@@
 <rectangle x1="-0.375" y1="5.625" x2="0.375" y2="6.375" layer="21"/>
 <rectangle x1="4.125" y1="5.625" x2="6.375" y2="6.375" layer="21"/>
-<rectangle x1="28.875" y1="5.625" x2="31.125" y2="6.375" layer="21"/>
+<rectangle x1="30.375" y1="5.625" x2="32.625" y2="6.375" layer="21"/>
 <rectangle x1="34.875" y1="5.625" x2="37.125" y2="6.375" layer="21"/>
 <rectangle x1="-0.375" y1="6.375" x2="0.375" y2="7.125" layer="21"/>
 <rectangle x1="4.125" y1="6.375" x2="6.375" y2="7.125" layer="21"/>
-<rectangle x1="28.875" y1="6.375" x2="31.125" y2="7.125" layer="21"/>
+<rectangle x1="30.375" y1="6.375" x2="32.625" y2="7.125" layer="21"/>
 <rectangle x1="34.875" y1="6.375" x2="37.125" y2="7.125" layer="21"/>
 <rectangle x1="-0.375" y1="7.125" x2="0.375" y2="7.875" layer="21"/>
 <rectangle x1="4.125" y1="7.125" x2="6.375" y2="7.875" layer="21"/>
-<rectangle x1="28.875" y1="7.125" x2="31.125" y2="7.875" layer="21"/>
+<rectangle x1="30.375" y1="7.125" x2="32.625" y2="7.875" layer="21"/>
 <rectangle x1="34.875" y1="7.125" x2="37.125" y2="7.875" layer="21"/>
 <rectangle x1="-0.375" y1="7.875" x2="0.375" y2="8.625" layer="21"/>
@@
 <rectangle x1="34.875" y1="29.625" x2="37.125" y2="30.375" layer="21"/>
 <rectangle x1="-0.375" y1="30.375" x2="0.375" y2="31.125" layer="21"/>
-<rectangle x1="4.125" y1="30.375" x2="6.375" y2="31.125" layer="21"/>
-<rectangle x1="28.875" y1="30.375" x2="31.125" y2="31.125" layer="21"/>
+<rectangle x1="4.125" y1="29.625" x2="6.375" y2="30.375" layer="21"/>
+<rectangle x1="30.375" y1="29.625" x2="32.625" y2="30.375" layer="21"/>
 <rectangle x1="34.875" y1="30.375" x2="37.125" y2="31.125" layer="21"/>
 <rectangle x1="-0.375" y1="31.125" x2="0.375" y2="31.875" layer="21"/>
-<rectangle x1="4.125" y1="31.125" x2="6.375" y2="31.875" layer="21"/>
-<rectangle x1="28.875" y1="31.125" x2="31.125" y2="31.875" layer="21"/>
+<rectangle x1="4.125" y1="30.375" x2="6.375" y2="31.125" layer="21"/>
+<rectangle x1="30.375" y1="30.375" x2="32.625" y2="31.125" layer="21"/>
 <rectangle x1="34.875" y1="31.125" x2="37.125" y2="31.875" layer="21"/>
 <rectangle x1="-0.375" y1="31.875" x2="0.375" y2="32.625" layer="21"/>
-<rectangle x1="4.125" y1="31.875" x2="6.375" y2="32.625" layer="21"/>
-<rectangle x1="28.875" y1="31.875" x2="31.125" y2="32.625" layer="21"/>
+<rectangle x1="4.125" y1="31.125" x2="6.375" y2="31.875" layer="21"/>
+<rectangle x1="30.375" y1="31.125" x2="32.625" y2="31.875" layer="21"/>
 <rectangle x1="34.875" y1="31.875" x2="37.125" y2="32.625" layer="21"/>
 <rectangle x1="-0.375" y1="32.625" x2="0.375" y2="33.375" layer="21"/>
@@
 <rectangle x1="-0.375" y1="34.125" x2="0.375" y2="34.875" layer="21"/>
 <rectangle x1="34.875" y1="34.125" x2="37.125" y2="34.875" layer="21"/>
+<rectangle x1="-0.375" y1="34.125" x2="1.875" y2="34.875" layer="21"/>
+<rectangle x1="34.875" y1="34.875" x2="37.125" y2="35.625" layer="21"/>
 <rectangle x1="-0.375" y1="34.875" x2="1.875" y2="35.625" layer="21"/>
-<rectangle x1="34.875" y1="34.875" x2="37.125" y2="35.625" layer="21"/>
-<rectangle x1="-0.375" y1="35.625" x2="1.875" y2="36.375" layer="21"/>
 <rectangle x1="34.875" y1="35.625" x2="37.125" y2="36.375" layer="21"/>
-<rectangle x1="-0.375" y1="36.375" x2="37.125" y2="37.125" layer="21"/>
+<rectangle x1="-0.375" y1="35.625" x2="37.125" y2="36.375" layer="21"/>
 <rectangle x1="11.625" y1="37.125" x2="23.625" y2="37.875" layer="21"/>
 <rectangle x1="11.625" y1="37.875" x2="23.625" y2="38.625" layer="21"/>
@@
 <attribute name="VALUE" x="23.7396" y="58.3804" size="1.27" layer="27" ratio="10" rot="R90"/>
 </element>
-<element name="BATTERY_1" library="Itead_BP_110825" package="BATTERY_1236_C" value="BATTERY_1236_C" x="28.86" y="19.04975" smashed="yes" rot="MR270"/>
+<element name="BATTERY_1" library="Itead_BP_110825" package="BATTERY_1236_C" value="BATTERY_1236_C" x="28.11" y="16.04975" smashed="yes" rot="MR270"/>
 </elements>
 <signals>
@@
 <contactref element="LED2" pad="K"/>
 <contactref element="LED1" pad="K"/>
-<wire x1="28.86" y1="19.04975" x2="18.75" y2="29.15975" width="0.8128" layer="1"/>
-<wire x1="18.75" y1="29.15975" x2="18.75" y2="51" width="0.8128" layer="1"/>
+<wire x1="28.11" y1="16.04975" x2="18.75" y2="27.65975" width="0.8128" layer="1"/>
+<wire x1="18.75" y1="27.65975" x2="18.75" y2="51" width="0.8128" layer="1"/>
 <wire x1="18.75" y1="51" x2="18" y2="51.75" width="0.8128" layer="1"/>
 <wire x1="18" y1="51.75" x2="18" y2="56.25" width="0.8128" layer="1"/>
@@
 <contactref element="LED2" pad="A"/>
 <contactref element="BATTERY_1" pad="-"/>
-<wire x1="8.54" y1="19.04975" x2="8.54975" y2="19.04975" width="0.8128" layer="1"/>
-<wire x1="8.54975" y1="19.04975" x2="17.25" y2="27.75" width="0.8128" layer="1"/>
+<wire x1="7.79" y1="16.04975" x2="10.04975" y2="19.04975" width="0.8128" layer="1"/>
+<wire x1="10.04975" y1="19.04975" x2="17.25" y2="27.75" width="0.8128" layer="1"/>
 <wire x1="17.25" y1="27.75" x2="17.25" y2="49.5" width="0.8128" layer="1"/>
 <via x="17.25" y="49.5" extent="1-16" drill="1" shape="octagon"/>
@@
 </board>
 </drawing>
-<compatibility>
-<note version="6.3" minversion="6.2.2" severity="warning">
-Since Version 6.2.2 text objects can contain more than one line,
-which will not be processed correctly with this version.
-</note>
-</compatibility>
 </eagle>
